File: TPIC/Microcontroller.kicad_sch (KiCad schematic)
At the start: 0 parts

Commit message: did some work to the schematic reagrding the MCU
Parts:
- added C3, C4: 10p, symbol Device:C
- added IC3: STM32G474QET6, QFP40P1600X1600X160-128N, symbol STM32G474QET6:STM32G474QET6
- added R1: R, symbol Device:R
- added Y1: ECS-80-10-33-CGN-TR3, ECS801033CGNTR3, symbol ECS-80-10-33-CGN-TR3:ECS-80-10-33-CGN-TR3
Connections:
- new net: C3.1, IC3.19 (PF0-OSC_IN), Y1.1 (IN/OUT)
- new net: C4.1, R1.2, Y1.3 (OUT/IN)
- new net: IC3.20 (PF1-OSC_OUT), R1.1
- new net GND: C3.2, C4.2, Y1.2 (GND_1), Y1.4 (GND_2)
Other:
- note added: "Vdd kobles til 3V3. VBAT kobles til 3V3. Vdda kobles til 3V3 med ekstra filtrering. Vss kobles til GND. VSSA kobles til GND"
