File: TPIC/TPIC.kicad_pcb (KiCad board)
At the start: 2 copper layers, 4 parts, among them IC1 7461383, IC2 7461383

Commit message: did some work to the schematic reagrding the MCU
Parts:
- added IC3: STM32G474QET6, STM32MCU:QFP40P1600X1600X160-128N, F.Cu at (92.3, 43.8)
- added Y1: ECS-80-10-33-CGN-TR3, 8MHzCrystal:ECS801033CGNTR3, F.Cu at (86.4, 56.0)
Connections:
- net Net-(C1-+) renamed /Connectors/Vin+
- net Net-(C1--) renamed /Connectors/Vin-
